File: Hardware/PCB/Custom Keyboard PCB V1/Custom Keyboard PCB V1/Custom Keyboard PCB V1.kicad_pcb (KiCad board)
At the start: 2 copper layers, 175 parts, among them J1 Conn_01x04, J2 Conn_01x01, J3 Conn_01x01, J4 Conn_01x01, J5 Conn_01x01, SW1 SW_Push, SW10 SW_Push, SW11 SW_Push, SW12 SW_Push, SW13 SW_Push, SW14 SW_Push, SW15 SW_Push, SW16 SW_Push, SW17 SW_Push, SW18 SW_Push, SW19 SW_Push, SW2 SW_Push, SW20 SW_Push, SW21 SW_Push, SW22 SW_Push, SW23 SW_Push, SW24 SW_Push, SW25 SW_Push, SW26 SW_Push, SW27 SW_Push, SW28 SW_Push, SW29 SW_Push, SW3 SW_Push, SW30 SW_Push, SW31 SW_Push, SW32 SW_Push, SW33 SW_Push, SW34 SW_Push, SW35 SW_Push, SW36 SW_Push, SW37 SW_Push, SW38 SW_Push, SW39 SW_Push, SW4 SW_Push, SW40 SW_Push, SW41 SW_Push, SW42 SW_Push, SW43 SW_Push, SW44 SW_Push, SW45 SW_Push, SW46 SW_Push, SW47 SW_Push, SW48 SW_Push, SW49 SW_Push, SW5 SW_Push, SW50 SW_Push, SW51 SW_Push, SW52 SW_Push, SW53 SW_Push, SW54 SW_Push, SW55 SW_Push, SW56 SW_Push, SW57 SW_Push, SW58 SW_Push, SW59 SW_Push, SW6 SW_Push, SW60 SW_Push, SW61 SW_Push, SW62 SW_Push, SW63 SW_Push, SW64 SW_Push, SW65 SW_Push, SW66 SW_Push, SW67 SW_Push, SW68 SW_Push, SW69 SW_Push, SW7 SW_Push, SW70 SW_Push, SW71 SW_Push, SW72 SW_Push, SW73 SW_Push, SW74 SW_Push, SW75 SW_Push, SW76 SW_Push, SW77 SW_Push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

Commit message: Hopefully fix
Parts:
- D18, D19, D20, D21, D22, D23, D24, D25, D26, D27, D28, D29, D30, D31, D32, D33, D34, D35, D36, D37, D38, D39, D40, D41, D42, D43, D44, D45, D46, D47, D48, D49, D50, D51, D52, D53, D54, D55, D56, D57, D58, D59, D60, D61, D62, D63, D64, D65, D66, D67, D68, D69, D70, D71, D72, D73, D74, D75, D76, D77, D78, D79, D80: moved to B.Cu
- moved D69 364.0 mm to (-527.2, -210.8)
- moved D35 364.0 mm to (-548.0, -210.8)
- moved D52 364.0 mm to (-537.6, -210.8)
- moved D18 364.0 mm to (-558.4, -210.8)
- moved D70 361.8 mm to (-527.2, -214.2)
- moved D36 361.8 mm to (-548.0, -214.2)
- moved D53 361.8 mm to (-537.6, -214.2)
- moved D19 361.8 mm to (-558.4, -214.2)
- moved D71 359.8 mm to (-527.2, -217.5)
- moved D37 359.8 mm to (-548.0, -217.5)
- moved D54 359.8 mm to (-537.6, -217.5)
- moved D20 359.8 mm to (-558.4, -217.5)
- moved D38 357.9 mm to (-548.0, -220.8)
- moved D55 357.9 mm to (-537.6, -220.8)
- moved D72 357.9 mm to (-527.2, -220.8)
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