File: Hardware/PCB/Custom Keyboard PCB V1/Custom Keyboard PCB V1/Custom Keyboard PCB V1.kicad_pcb (KiCad board)
At the start: 2 copper layers, 1 part, among them U1 WeMos_S3_mini

Commit message: uhhhhhhhhhhhhhhhhhhhhhhhhhhhhhhhhhhhhh
Parts:
- added D1: 1N4148, Diode_SMD:D_MiniMELF_Handsoldering, F.Cu at (38.1, 38.1)
- added D10: 1N4148, Diode_SMD:D_MiniMELF_Handsoldering, F.Cu at (247.7, 38.1)
- added D11: 1N4148, Diode_SMD:D_MiniMELF_Handsoldering, F.Cu at (266.7, 38.1)
- added D12: 1N4148, Diode_SMD:D_MiniMELF_Handsoldering, F.Cu at (285.8, 38.1)
- added D13: 1N4148, Diode_SMD:D_MiniMELF_Handsoldering, F.Cu at (304.8, 38.1)
- added D14: 1N4148, Diode_SMD:D_MiniMELF_Handsoldering, F.Cu at (38.1, 66.7)
- added D15: 1N4148, Diode_SMD:D_MiniMELF_Handsoldering, F.Cu at (57.1, 66.7)
- added D16: 1N4148, Diode_SMD:D_MiniMELF_Handsoldering, F.Cu at (76.2, 66.7)
- added D17: 1N4148, Diode_SMD:D_MiniMELF_Handsoldering, F.Cu at (95.2, 66.7)
- added D18: 1N4148, Diode_SMD:D_MiniMELF_Handsoldering, F.Cu at (114.3, 66.7)
- added D19: 1N4148, Diode_SMD:D_MiniMELF_Handsoldering, F.Cu at (133.3, 66.7)
- added D2: 1N4148, Diode_SMD:D_MiniMELF_Handsoldering, F.Cu at (76.2, 38.1)
- added D20: 1N4148, Diode_SMD:D_MiniMELF_Handsoldering, F.Cu at (152.4, 66.7)
- added D21: 1N4148, Diode_SMD:D_MiniMELF_Handsoldering, F.Cu at (171.4, 66.7)
- added D22: 1N4148, Diode_SMD:D_MiniMELF_Handsoldering, F.Cu at (190.5, 66.7)
- added D23: 1N4148, Diode_SMD:D_MiniMELF_Handsoldering, F.Cu at (209.6, 66.7)
- added D24: 1N4148, Diode_SMD:D_MiniMELF_Handsoldering, F.Cu at (228.6, 66.7)
- added D25: 1N4148, Diode_SMD:D_MiniMELF_Handsoldering, F.Cu at (247.7, 66.7)
- added D26: 1N4148, Diode_SMD:D_MiniMELF_Handsoldering, F.Cu at (266.7, 66.7)
- added D27: 1N4148, Diode_SMD:D_MiniMELF_Handsoldering, F.Cu at (295.3, 66.7)
- added D28: 1N4148, Diode_SMD:D_MiniMELF_Handsoldering, F.Cu at (42.9, 85.7)
- added D29: 1N4148, Diode_SMD:D_MiniMELF_Handsoldering, F.Cu at (66.7, 85.7)
- added D3: 1N4148, Diode_SMD:D_MiniMELF_Handsoldering, F.Cu at (95.2, 38.1)
- added D30: 1N4148, Diode_SMD:D_MiniMELF_Handsoldering, F.Cu at (85.7, 85.7)
- added D31: 1N4148, Diode_SMD:D_MiniMELF_Handsoldering, F.Cu at (104.8, 85.7)
- added D32: 1N4148, Diode_SMD:D_MiniMELF_Handsoldering, F.Cu at (123.8, 85.7)
- added D33: 1N4148, Diode_SMD:D_MiniMELF_Handsoldering, F.Cu at (142.9, 85.7)
- added D34: 1N4148, Diode_SMD:D_MiniMELF_Handsoldering, F.Cu at (161.9, 85.7)
- added D35: 1N4148, Diode_SMD:D_MiniMELF_Handsoldering, F.Cu at (181.0, 85.7)
- added D36: 1N4148, Diode_SMD:D_MiniMELF_Handsoldering, F.Cu at (200.0, 85.7)
- added D37: 1N4148, Diode_SMD:D_MiniMELF_Handsoldering, F.Cu at (219.1, 85.7)
- added D38: 1N4148, Diode_SMD:D_MiniMELF_Handsoldering, F.Cu at (238.1, 85.7)
- added D39: 1N4148, Diode_SMD:D_MiniMELF_Handsoldering, F.Cu at (257.2, 85.7)
- added D4: 1N4148, Diode_SMD:D_MiniMELF_Handsoldering, F.Cu at (114.3, 38.1)
- added D40: 1N4148, Diode_SMD:D_MiniMELF_Handsoldering, F.Cu at (276.2, 85.7)
- added D41: 1N4148, Diode_SMD:D_MiniMELF_Handsoldering, F.Cu at (300.0, 85.7)
- added D42: 1N4148, Diode_SMD:D_MiniMELF_Handsoldering, F.Cu at (45.2, 104.8)
- added D43: 1N4148, Diode_SMD:D_MiniMELF_Handsoldering, F.Cu at (71.4, 104.8)
- added D44: 1N4148, Diode_SMD:D_MiniMELF_Handsoldering, F.Cu at (90.5, 104.8)
- added D45: 1N4148, Diode_SMD:D_MiniMELF_Handsoldering, F.Cu at (109.5, 104.8)
- added D46: 1N4148, Diode_SMD:D_MiniMELF_Handsoldering, F.Cu at (128.6, 104.8)
- added D47: 1N4148, Diode_SMD:D_MiniMELF_Handsoldering, F.Cu at (147.6, 104.8)
- added D48: 1N4148, Diode_SMD:D_MiniMELF_Handsoldering, F.Cu at (166.7, 104.8)
- added D49: 1N4148, Diode_SMD:D_MiniMELF_Handsoldering, F.Cu at (185.7, 104.8)
- added D5: 1N4148, Diode_SMD:D_MiniMELF_Handsoldering, F.Cu at (133.3, 38.1)
- added D50: 1N4148, Diode_SMD:D_MiniMELF_Handsoldering, F.Cu at (204.8, 104.8)
- added D51: 1N4148, Diode_SMD:D_MiniMELF_Handsoldering, F.Cu at (223.8, 104.8)
- added D52: 1N4148, Diode_SMD:D_MiniMELF_Handsoldering, F.Cu at (242.9, 104.8)
- added D53: 1N4148, Diode_SMD:D_MiniMELF_Handsoldering, F.Cu at (261.9, 104.8)
- added D54: 1N4148, Diode_SMD:D_MiniMELF_Handsoldering, F.Cu at (292.9, 104.8)
- added D55: 1N4148, Diode_SMD:D_MiniMELF_Handsoldering, F.Cu at (50.0, 123.8)
- added D56: 1N4148, Diode_SMD:D_MiniMELF_Handsoldering, F.Cu at (81.0, 123.8)
- added D57: 1N4148, Diode_SMD:D_MiniMELF_Handsoldering, F.Cu at (100.0, 123.8)
- added D58: 1N4148, Diode_SMD:D_MiniMELF_Handsoldering, F.Cu at (119.1, 123.8)
- added D59: 1N4148, Diode_SMD:D_MiniMELF_Handsoldering, F.Cu at (138.1, 123.8)
- added D6: 1N4148, Diode_SMD:D_MiniMELF_Handsoldering, F.Cu at (161.9, 38.1)
- added D60: 1N4148, Diode_SMD:D_MiniMELF_Handsoldering, F.Cu at (157.2, 123.8)
- added D61: 1N4148, Diode_SMD:D_MiniMELF_Handsoldering, F.Cu at (176.2, 123.8)
- added D62: 1N4148, Diode_SMD:D_MiniMELF_Handsoldering, F.Cu at (195.3, 123.8)
- added D63: 1N4148, Diode_SMD:D_MiniMELF_Handsoldering, F.Cu at (214.3, 123.8)
- added D64: 1N4148, Diode_SMD:D_MiniMELF_Handsoldering, F.Cu at (233.4, 123.8)
- added D65: 1N4148, Diode_SMD:D_MiniMELF_Handsoldering, F.Cu at (252.4, 123.8)
- added D66: 1N4148, Diode_SMD:D_MiniMELF_Handsoldering, F.Cu at (288.1, 123.8)
- added D67: 1N4148, Diode_SMD:D_MiniMELF_Handsoldering, F.Cu at (328.6, 123.8)
- added D68: 1N4148, Diode_SMD:D_MiniMELF_Handsoldering, F.Cu at (347.7, 123.8)
- added D69: 1N4148, Diode_SMD:D_MiniMELF_Handsoldering, F.Cu at (366.7, 123.8)
- added D7: 1N4148, Diode_SMD:D_MiniMELF_Handsoldering, F.Cu at (181.0, 38.1)
- added D70: 1N4148, Diode_SMD:D_MiniMELF_Handsoldering, F.Cu at (40.5, 142.9)
- added D71: 1N4148, Diode_SMD:D_MiniMELF_Handsoldering, F.Cu at (64.3, 142.9)
- added D72: 1N4148, Diode_SMD:D_MiniMELF_Handsoldering, F.Cu at (88.1, 142.9)
- added D73: 1N4148, Diode_SMD:D_MiniMELF_Handsoldering, F.Cu at (159.5, 142.9)
- added D74: 1N4148, Diode_SMD:D_MiniMELF_Handsoldering, F.Cu at (231.0, 142.9)
- added D75: 1N4148, Diode_SMD:D_MiniMELF_Handsoldering, F.Cu at (254.8, 142.9)
- added D76: 1N4148, Diode_SMD:D_MiniMELF_Handsoldering, F.Cu at (278.6, 142.9)
- added D77: 1N4148, Diode_SMD:D_MiniMELF_Handsoldering, F.Cu at (302.4, 142.9)
- added D78: 1N4148, Diode_SMD:D_MiniMELF_Handsoldering, F.Cu at (328.6, 142.9)
- added D79: 1N4148, Diode_SMD:D_MiniMELF_Handsoldering, F.Cu at (347.7, 142.9)
- added D8: 1N4148, Diode_SMD:D_MiniMELF_Handsoldering, F.Cu at (200.0, 38.1)
- added D80: 1N4148, Diode_SMD:D_MiniMELF_Handsoldering, F.Cu at (366.7, 142.9)
- added D9: 1N4148, Diode_SMD:D_MiniMELF_Handsoldering, F.Cu at (219.1, 38.1)
- added J1: Conn_01x04, Wireless Keyboard:OLED_SSD1306_I2C_0.96, F.Cu at (-423.5, 133.8)
- added J2: Conn_01x01, Connector_PinHeader_2.54mm:PinHeader_1x01_P2.54mm_Vertical, F.Cu at (-403.2, 149.1)
- added J3: Conn_01x01, Connector_PinHeader_2.54mm:PinHeader_1x01_P2.54mm_Vertical, F.Cu at (-403.2, 153.7)
- added J4: Conn_01x01, Connector_PinHeader_2.54mm:PinHeader_1x01_P2.54mm_Vertical, F.Cu at (-403.2, 158.3)
- added J5: Conn_01x01, Connector_PinHeader_2.54mm:PinHeader_1x01_P2.54mm_Vertical, F.Cu at (-403.2, 162.8)
- added R1: 5k, Resistor_THT:R_Axial_DIN0204_L3.6mm_D1.6mm_P5.08mm_Horizontal, F.Cu at (-399.4, 148.4)
- added R2: 5k, Resistor_THT:R_Axial_DIN0204_L3.6mm_D1.6mm_P5.08mm_Horizontal, F.Cu at (-399.4, 151.5)
- added R3: 5k, Resistor_THT:R_Axial_DIN0204_L3.6mm_D1.6mm_P5.08mm_Horizontal, F.Cu at (-399.4, 154.7)
- added S1: MX_stab, PCM_marbastlib-mx:STAB_MX_P_2u, F.Cu at (38.1, 38.1)
- added S2: MX_stab, PCM_marbastlib-mx:STAB_MX_P_2u, F.Cu at (76.2, 38.1)
- added S3: MX_stab, PCM_marbastlib-mx:STAB_MX_P_2u, F.Cu at (95.2, 38.1)
- added S4: MX_stab, PCM_marbastlib-mx:STAB_MX_P_2u, F.Cu at (114.3, 38.1)
- added S5: MX_stab, PCM_marbastlib-mx:STAB_MX_P_6.25u, F.Cu at (133.3, 38.1)
- added SW1: SW_Push, PCM_marbastlib-mx:SW_MX_1u, F.Cu at (38.1, 38.1)
- added SW10: SW_Push, PCM_marbastlib-mx:SW_MX_1u, F.Cu at (247.7, 38.1)
- added SW11: SW_Push, PCM_marbastlib-mx:SW_MX_1u, F.Cu at (266.7, 38.1)
- added SW12: SW_Push, PCM_marbastlib-mx:SW_MX_1u, F.Cu at (285.8, 38.1)
- added SW13: SW_Push, PCM_marbastlib-mx:SW_MX_1u, F.Cu at (304.8, 38.1)
- added SW14: SW_Push, PCM_marbastlib-mx:SW_MX_1u, F.Cu at (38.1, 66.7)
- added SW15: SW_Push, PCM_marbastlib-mx:SW_MX_1u, F.Cu at (57.1, 66.7)
- added SW16: SW_Push, PCM_marbastlib-mx:SW_MX_1u, F.Cu at (76.2, 66.7)
- added SW17: SW_Push, PCM_marbastlib-mx:SW_MX_1u, F.Cu at (95.2, 66.7)
- added SW18: SW_Push, PCM_marbastlib-mx:SW_MX_1u, F.Cu at (114.3, 66.7)
- added SW19: SW_Push, PCM_marbastlib-mx:SW_MX_1u, F.Cu at (133.3, 66.7)
- added SW2: SW_Push, PCM_marbastlib-mx:SW_MX_1u, F.Cu at (76.2, 38.1)
- added SW20: SW_Push, PCM_marbastlib-mx:SW_MX_1u, F.Cu at (152.4, 66.7)
- added SW21: SW_Push, PCM_marbastlib-mx:SW_MX_1u, F.Cu at (171.4, 66.7)
- added SW22: SW_Push, PCM_marbastlib-mx:SW_MX_1u, F.Cu at (190.5, 66.7)
- added SW23: SW_Push, PCM_marbastlib-mx:SW_MX_1u, F.Cu at (209.6, 66.7)
- added SW24: SW_Push, PCM_marbastlib-mx:SW_MX_1u, F.Cu at (228.6, 66.7)
- added SW25: SW_Push, PCM_marbastlib-mx:SW_MX_1u, F.Cu at (247.7, 66.7)
- added SW26: SW_Push, PCM_marbastlib-mx:SW_MX_1u, F.Cu at (266.7, 66.7)
- added SW27: SW_Push, PCM_marbastlib-mx:SW_MX_1u, F.Cu at (295.3, 66.7)
- added SW28: SW_Push, PCM_marbastlib-mx:SW_MX_1u, F.Cu at (42.9, 85.7)
- added SW29: SW_Push, PCM_marbastlib-mx:SW_MX_1u, F.Cu at (66.7, 85.7)
- added SW3: SW_Push, PCM_marbastlib-mx:SW_MX_1u, F.Cu at (95.2, 38.1)
- added SW30: SW_Push, PCM_marbastlib-mx:SW_MX_1u, F.Cu at (85.7, 85.7)
- added SW31: SW_Push, PCM_marbastlib-mx:SW_MX_1u, F.Cu at (104.8, 85.7)
- added SW32: SW_Push, PCM_marbastlib-mx:SW_MX_1u, F.Cu at (123.8, 85.7)
- added SW33: SW_Push, PCM_marbastlib-mx:SW_MX_1u, F.Cu at (142.9, 85.7)
- added SW34: SW_Push, PCM_marbastlib-mx:SW_MX_1u, F.Cu at (161.9, 85.7)
- added SW35: SW_Push, PCM_marbastlib-mx:SW_MX_1u, F.Cu at (181.0, 85.7)
- added SW36: SW_Push, PCM_marbastlib-mx:SW_MX_1u, F.Cu at (200.0, 85.7)
- added SW37: SW_Push, PCM_marbastlib-mx:SW_MX_1u, F.Cu at (219.1, 85.7)
- added SW38: SW_Push, PCM_marbastlib-mx:SW_MX_1u, F.Cu at (238.1, 85.7)
- added SW39: SW_Push, PCM_marbastlib-mx:SW_MX_1u, F.Cu at (257.2, 85.7)
- added SW4: SW_Push, PCM_marbastlib-mx:SW_MX_1u, F.Cu at (114.3, 38.1)
- added SW40: SW_Push, PCM_marbastlib-mx:SW_MX_1u, F.Cu at (276.2, 85.7)
- added SW41: SW_Push, PCM_marbastlib-mx:SW_MX_1u, F.Cu at (300.0, 85.7)
- added SW42: SW_Push, PCM_marbastlib-mx:SW_MX_1u, F.Cu at (45.2, 104.8)
- added SW43: SW_Push, PCM_marbastlib-mx:SW_MX_1u, F.Cu at (71.4, 104.8)
- added SW44: SW_Push, PCM_marbastlib-mx:SW_MX_1u, F.Cu at (90.5, 104.8)
- added SW45: SW_Push, PCM_marbastlib-mx:SW_MX_1u, F.Cu at (109.5, 104.8)
- added SW46: SW_Push, PCM_marbastlib-mx:SW_MX_1u, F.Cu at (128.6, 104.8)
- added SW47: SW_Push, PCM_marbastlib-mx:SW_MX_1u, F.Cu at (147.6, 104.8)
- added SW48: SW_Push, PCM_marbastlib-mx:SW_MX_1u, F.Cu at (166.7, 104.8)
- added SW49: SW_Push, PCM_marbastlib-mx:SW_MX_1u, F.Cu at (185.7, 104.8)
- added SW5: SW_Push, PCM_marbastlib-mx:SW_MX_1u, F.Cu at (133.3, 38.1)
- added SW50: SW_Push, PCM_marbastlib-mx:SW_MX_1u, F.Cu at (204.8, 104.8)
- added SW51: SW_Push, PCM_marbastlib-mx:SW_MX_1u, F.Cu at (223.8, 104.8)
- added SW52: SW_Push, PCM_marbastlib-mx:SW_MX_1u, F.Cu at (242.9, 104.8)
- added SW53: SW_Push, PCM_marbastlib-mx:SW_MX_1u, F.Cu at (261.9, 104.8)
- added SW54: SW_Push, PCM_marbastlib-mx:SW_MX_1u, F.Cu at (292.9, 104.8)
- added SW55: SW_Push, PCM_marbastlib-mx:SW_MX_1u, F.Cu at (50.0, 123.8)
- added SW56: SW_Push, PCM_marbastlib-mx:SW_MX_1u, F.Cu at (81.0, 123.8)
- added SW57: SW_Push, PCM_marbastlib-mx:SW_MX_1u, F.Cu at (100.0, 123.8)
- added SW58: SW_Push, PCM_marbastlib-mx:SW_MX_1u, F.Cu at (119.1, 123.8)
- added SW59: SW_Push, PCM_marbastlib-mx:SW_MX_1u, F.Cu at (138.1, 123.8)
- added SW6: SW_Push, PCM_marbastlib-mx:SW_MX_1u, F.Cu at (161.9, 38.1)
- added SW60: SW_Push, PCM_marbastlib-mx:SW_MX_1u, F.Cu at (157.2, 123.8)
- added SW61: SW_Push, PCM_marbastlib-mx:SW_MX_1u, F.Cu at (176.2, 123.8)
- added SW62: SW_Push, PCM_marbastlib-mx:SW_MX_1u, F.Cu at (195.3, 123.8)
- added SW63: SW_Push, PCM_marbastlib-mx:SW_MX_1u, F.Cu at (214.3, 123.8)
- added SW64: SW_Push, PCM_marbastlib-mx:SW_MX_1u, F.Cu at (233.4, 123.8)
- added SW65: SW_Push, PCM_marbastlib-mx:SW_MX_1u, F.Cu at (252.4, 123.8)
- added SW66: SW_Push, PCM_marbastlib-mx:SW_MX_1u, F.Cu at (288.1, 123.8)
- added SW67: SW_Push, PCM_marbastlib-mx:SW_MX_1u, F.Cu at (328.6, 123.8)
- added SW68: SW_Push, PCM_marbastlib-mx:SW_MX_1u, F.Cu at (347.7, 123.8)
- added SW69: SW_Push, PCM_marbastlib-mx:SW_MX_1u, F.Cu at (366.7, 123.8)
- added SW7: SW_Push, PCM_marbastlib-mx:SW_MX_1u, F.Cu at (181.0, 38.1)
- added SW70: SW_Push, PCM_marbastlib-mx:SW_MX_1u, F.Cu at (40.5, 142.9)
- added SW71: SW_Push, PCM_marbastlib-mx:SW_MX_1u, F.Cu at (64.3, 142.9)
- added SW72: SW_Push, PCM_marbastlib-mx:SW_MX_1u, F.Cu at (88.1, 142.9)
- added SW73: SW_Push, PCM_marbastlib-mx:SW_MX_1u, F.Cu at (159.5, 142.9)
- added SW74: SW_Push, PCM_marbastlib-mx:SW_MX_1u, F.Cu at (231.0, 142.9)
- added SW75: SW_Push, PCM_marbastlib-mx:SW_MX_1u, F.Cu at (254.8, 142.9)
- added SW76: SW_Push, PCM_marbastlib-mx:SW_MX_1u, F.Cu at (278.6, 142.9)
- added SW77: SW_Push, PCM_marbastlib-mx:SW_MX_1u, F.Cu at (302.4, 142.9)
- added SW78: SW_Push, PCM_marbastlib-mx:SW_MX_1u, F.Cu at (328.6, 142.9)
- added SW79: SW_Push, PCM_marbastlib-mx:SW_MX_1u, F.Cu at (347.7, 142.9)
- added SW8: SW_Push, PCM_marbastlib-mx:SW_MX_1u, F.Cu at (200.0, 38.1)
- added SW80: SW_Push, PCM_marbastlib-mx:SW_MX_1u, F.Cu at (366.7, 142.9)
- added SW9: SW_Push, PCM_marbastlib-mx:SW_MX_1u, F.Cu at (219.1, 38.1)
- added SW_EC11: RotaryEncoder_Switch_MP, Rotary_Encoder:RotaryEncoder_Alps_EC11E-Switch_Vertical_H20mm_MountingHoles, F.Cu at (-403.4, 136.7)
- moved U1 442.6 mm to (-280.3, 80.8), turned to 0 degrees
Connections:
- U1 pad 1: /MCU_EN -> unconnected-(U1-EN-Pad1)
- U1 pad 11: /GPIO16 -> /COL15
- U1 pad 12: /GPIO18 -> /ROW3
- U1 pad 13: /GPIO35 -> /GPIO35(SDA)
- U1 pad 14: /GPIO36 -> /GPIO36(SCL)
- U1 pad 15: /GPIO44 -> /GPIO44_(EC11_B)
- U1 pad 16: /GPIO43 -> /GPIO43_(EC11_A)
- U1 pad 17: /GPIO01 -> /COL1
- U1 pad 18: /GPIO03 -> /COL2
- U1 pad 19: /GPIO05 -> /COL4
- U1 pad 2: /GPIO02 -> /COL3
- U1 pad 20: /GPIO06 -> /COL6
- U1 pad 21: /GPIO07 -> /COL8
- U1 pad 22: /GPIO08 -> /COL10
- U1 pad 23: /GPIO09 -> /COL13
- U1 pad 24: /GPIO14 -> /COL14
- U1 pad 25: /GPIO15 -> /ROW1
- U1 pad 27: /GPIO17 -> /ROW2
- U1 pad 28: /GPIO21 -> /ROW4
- U1 pad 29: /GPIO34 -> /ROW5
- U1 pad 3: /GPIO04 -> /COL5
- U1 pad 30: /GPIO38 -> /ROW6
- U1 pad 31: /GPIO37 -> unconnected-(U1-GPIO37-Pad31)
- U1 pad 32: /GPIO33 -> unconnected-(U1-GPIO33-Pad32)
- U1 pad 4: /GPIO12 -> /COL7
- U1 pad 5: /GPIO13 -> /COL9
- U1 pad 6: /GPIO11 -> /COL11
- U1 pad 7: /GPIO10 -> /COL12
Routing:
- net Net-(D54-A): track 0.00 -> 25.8 mm
- net Net-(D79-A): track 0.00 -> 25.8 mm
- net Net-(D78-A): track 0.00 -> 25.8 mm
- net Net-(D41-A): track 0.00 -> 25.8 mm
- net Net-(D40-A): track 0.00 -> 25.8 mm
- net Net-(D39-A): track 0.00 -> 25.8 mm
- net Net-(D13-A): track 0.00 -> 25.8 mm
- net Net-(D66-A): track 0.00 -> 25.8 mm
- net Net-(D68-A): track 0.00 -> 25.8 mm
- net Net-(D67-A): track 0.00 -> 25.8 mm
- net Net-(D72-A): track 0.00 -> 25.8 mm
- net Net-(D71-A): track 0.00 -> 25.8 mm
- net Net-(D51-A): track 0.00 -> 25.8 mm
- net Net-(D50-A): track 0.00 -> 25.8 mm
- net Net-(D49-A): track 0.00 -> 25.8 mm
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
Commit message: vgcjyxurcuygvuhj
Parts:
- D1, D10, D11, D12, D13, D14, D15, D16, D17, D2, D3, D4, D5, D6, D7, D8, D9: moved to B.Cu
- moved D13 843.5 mm to (-496.8, -224.4), turned to 180 degrees
- moved D12 826.5 mm to (-496.8, -227.8), turned to 180 degrees
- moved D11 809.6 mm to (-496.8, -231.1), turned to 180 degrees
- moved SW13 799.5 mm to (-438.1, -257.2)
- moved D10 792.8 mm to (-496.8, -234.5), turned to 180 degrees
- moved D9 767.2 mm to (-496.8, -237.8), turned to 180 degrees
- moved D8 750.7 mm to (-496.8, -241.1), turned to 180 degrees
- moved SW11 739.3 mm to (-447.7, -152.4)
- moved SW12 734.7 mm to (-423.9, -152.4)
- moved D7 734.4 mm to (-496.8, -244.5), turned to 180 degrees
- moved D69 714.0 mm to (-183.7, -331.1)
- moved SW10 712.5 mm to (-433.4, -171.4)
- moved SW27 712.5 mm to (-376.2, -171.4)
- moved D80 702.9 mm to (-183.7, -294.3)
- moved SW26 701.3 mm to (-385.8, -190.5)
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Routing:
- net Net-(D54-A): track 25.8 -> 0.00 mm
- net Net-(D79-A): track 25.8 -> 0.00 mm
- net Net-(D78-A): track 25.8 -> 0.00 mm
- net Net-(D41-A): track 25.8 -> 0.00 mm
- net Net-(D40-A): track 25.8 -> 0.00 mm
- net Net-(D39-A): track 25.8 -> 0.00 mm
- net Net-(D13-A): track 25.8 -> 0.00 mm
- net Net-(D66-A): track 25.8 -> 0.00 mm
- net Net-(D68-A): track 25.8 -> 0.00 mm
- net Net-(D67-A): track 25.8 -> 0.00 mm
- net Net-(D72-A): track 25.8 -> 0.00 mm
- net Net-(D71-A): track 25.8 -> 0.00 mm
- net Net-(D51-A): track 25.8 -> 0.00 mm
- net Net-(D50-A): track 25.8 -> 0.00 mm
- net Net-(D49-A): track 25.8 -> 0.00 mm
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
Commit message: might be broken
Parts:
- D1, D10, D11, D12, D13, D14, D15, D16, D17, D2, D3, D4, D5, D6, D7, D8, D9: moved to F.Cu
- moved D13 843.5 mm to (304.8, 38.1), turned to 0 degrees
- moved D12 826.5 mm to (285.8, 38.1), turned to 0 degrees
- moved D11 809.6 mm to (266.7, 38.1), turned to 0 degrees
- moved SW13 799.5 mm to (304.8, 38.1)
- moved S3 796.1 mm to (295.3, 66.7)
- moved D10 792.8 mm to (247.7, 38.1), turned to 0 degrees
- moved D9 767.2 mm to (219.1, 38.1), turned to 0 degrees
- moved D8 750.7 mm to (200.0, 38.1), turned to 0 degrees
- moved SW11 739.3 mm to (266.7, 38.1)
- moved SW12 734.7 mm to (285.8, 38.1)
- moved D7 734.4 mm to (181.0, 38.1), turned to 0 degrees
- moved D69 714.0 mm to (366.7, 123.8)
- moved SW10 712.5 mm to (247.7, 38.1)
- moved SW27 712.5 mm to (295.3, 66.7)
- moved D80 702.9 mm to (366.7, 142.9)
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Connections:
- U1 pad 11: /COL15 -> /COL2
- U1 pad 12: /ROW3 -> /COL4
- U1 pad 15: /GPIO44_(EC11_B) -> /COL8
- U1 pad 16: /GPIO43_(EC11_A) -> /COL10
- U1 pad 17: /COL1 -> /COL12
- U1 pad 18: /COL2 -> /COL13
- U1 pad 19: /COL4 -> /COL15
- U1 pad 2: /COL3 -> /COL14
- U1 pad 20: /COL6 -> /ROW2
- U1 pad 21: /COL8 -> /ROW4
- U1 pad 22: /COL10 -> /ROW6
- U1 pad 23: /COL13 -> /GPIO44_(EC11_B)
- U1 pad 24: /COL14 -> unconnected-(U1-GPIO14-Pad24)
- U1 pad 25: /ROW1 -> /COL1
- U1 pad 27: /ROW2 -> /COL3
- U1 pad 28: /ROW4 -> /COL5
- U1 pad 29: /ROW5 -> /COL6
- U1 pad 3: /COL5 -> /ROW1
- U1 pad 30: /ROW6 -> /COL7
- U1 pad 31: unconnected-(U1-GPIO37-Pad31) -> /COL9
- U1 pad 32: unconnected-(U1-GPIO33-Pad32) -> /COL11
- U1 pad 4: /COL7 -> /ROW3
- U1 pad 5: /COL9 -> /ROW5
- U1 pad 6: /COL11 -> unconnected-(U1-GPIO11-Pad6)
- U1 pad 7: /COL12 -> /GPIO43_(EC11_A)
Routing:
- net Net-(D54-A): track 0.00 -> 25.8 mm
- net Net-(D79-A): track 0.00 -> 25.8 mm
- net Net-(D78-A): track 0.00 -> 25.8 mm
- net Net-(D41-A): track 0.00 -> 25.8 mm
- net Net-(D40-A): track 0.00 -> 25.8 mm
- net Net-(D39-A): track 0.00 -> 25.8 mm
- net Net-(D13-A): track 0.00 -> 25.8 mm
- net Net-(D66-A): track 0.00 -> 25.8 mm
- net Net-(D68-A): track 0.00 -> 25.8 mm
- net Net-(D67-A): track 0.00 -> 25.8 mm
- net Net-(D72-A): track 0.00 -> 25.8 mm
- net Net-(D71-A): track 0.00 -> 25.8 mm
- net Net-(D51-A): track 0.00 -> 25.8 mm
- net Net-(D50-A): track 0.00 -> 25.8 mm
- net Net-(D49-A): track 0.00 -> 25.8 mm
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Other:
- board outline added: 367.3 x 134 mm

Commit message: i guess maybe not broken
Parts:
- D1, D10, D11, D12, D13, D14, D15, D16, D17, D18, D19, D2, D20, D21, D22, D23, D24, D25, D26, D27, D28, D29, D3, D30, D31, D32, D33, D34, D35, D36, D37, D38, D39, D4, D40, D41, D42, D43, D44, D45, D46, D47, D48, D49, D5, D50, D51, D52, D53, D54, D55, D56, D57, D58, D59, D6, D60, D61, D62, D63, D64, D65, D66, D67, D68, D69, D7, D70, D71, D72, D73, D74, D75, D76, D77, D78, D79, D8, D80, D9: moved to B.Cu
- moved SW13 365.1 mm to (12.2, -180.3)
- moved D13 362.2 mm to (12.2, -175.3)
- moved SW70 350.9 mm to (231.2, -151.7)
- moved S3 348.8 mm to (-14.0, -94.5)
- moved D70 346.8 mm to (231.3, -146.7)
- moved SW55 332.2 mm to (183.6, -180.3)
- moved S1 329.8 mm to (231.2, -151.7)
- moved SW69 329.2 mm to (240.8, -180.3)
- moved D55 327.6 mm to (183.6, -175.3)
- moved SW71 324.6 mm to (236.0, -132.7)
- moved D69 324.5 mm to (240.8, -175.3)
- moved D71 319.4 mm to (234.1, -127.7)
- moved SW66 311.3 mm to (221.7, -180.3)
- moved D66 306.4 mm to (221.7, -175.3)
- moved SW61 305.2 mm to (202.7, -180.3)
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Connections:
- U1 pad 11: /COL2 -> /COL1
- U1 pad 25: /COL1 -> /COL2
Routing:
- net Net-(D54-A): track 25.8 -> 0.00 mm
- net Net-(D79-A): track 25.8 -> 0.00 mm
- net Net-(D78-A): track 25.8 -> 0.00 mm
- net Net-(D41-A): track 25.8 -> 0.00 mm
- net Net-(D40-A): track 25.8 -> 0.00 mm
- net Net-(D39-A): track 25.8 -> 0.00 mm
- net Net-(D13-A): track 25.8 -> 0.00 mm
- net Net-(D66-A): track 25.8 -> 0.00 mm
- net Net-(D68-A): track 25.8 -> 0.00 mm
- net Net-(D67-A): track 25.8 -> 0.00 mm
- net Net-(D72-A): track 25.8 -> 0.00 mm
- net Net-(D71-A): track 25.8 -> 0.00 mm
- net Net-(D51-A): track 25.8 -> 0.00 mm
- net Net-(D50-A): track 25.8 -> 0.00 mm
- net Net-(D49-A): track 25.8 -> 0.00 mm
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Other:
- board size 367.3 x 134 mm -> 360.5 x 131.8 mm

Commit message: uhhhhhhhhhhhhhhhhh
Parts:
- moved J2 70.8 mm to (296.4, -115.5), turned to 90 degrees
- moved J3 67.6 mm to (301.0, -115.5), turned to 90 degrees
- moved J4 64.8 mm to (305.6, -115.5), turned to 90 degrees
- moved J5 62.6 mm to (310.2, -115.5), turned to 90 degrees
- moved J1 18.7 mm to (269.6, -130.6)
- moved R1 8.90 mm to (265.7, -188.4)
- moved R3 8.90 mm to (270.7, -171.9)
- moved SW_EC11 8.90 mm to (260.8, -182.6)
- moved R2 8.90 mm to (260.3, -171.9)
- moved D71 1.95 mm to (236.0, -127.6)
- turned D14 to 0 degrees
Routing:
- net /ROW4: track 0.00 -> 648.5 mm
- net /ROW5: track 0.00 -> 640.5 mm
- net /ROW3: track 0.00 -> 604.1 mm
- net /ROW2: track 0.00 -> 586.8 mm
- net /ROW6: track 0.00 -> 583.1 mm
- net /ROW1: track 0.00 -> 581.9 mm
- net /COL1: track 0.00 -> 469.2 mm
- net /COL2: track 0.00 -> 468.1 mm
- net /COL3: track 0.00 -> 409.4 mm
- net /COL4: track 0.00 -> 379.1 mm
- net /COL6: track 0.00 -> 367.7 mm
- net /COL5: track 0.00 -> 364.2 mm
- net /COL7: track 0.00 -> 323.9 mm
- net /COL8: track 0.00 -> 302.3 mm
- net /COL11: track 0.00 -> 289.6 mm, vias 0 -> 1
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- added copper zone on B.Cu, net GND
- added copper zone on F.Cu, net GND
Other:
- outline, holes or cut-outs redrawn
